File: Schematic-and-Board/MP-Tracker.sch (KiCad schematic (older format))
At the start: 69 parts, among them P1 DIL10, Q1 BC817-40, Q2 IRFR5303, Q3 BC817-40, Q4 IRFR5303, U1 MC34063, U2 TL082, U3 ATMEGA8-AI, U4 MC78L033, X1 3.6864MHz

Commit message: New major revision of schematic. The most notable changes: Added three 3-step R/C filters to cancel noise from uC PWM and for current measurement. Switched from TL081 to MC4558 dual-OP-amp. (Better performance, cheaper, pin-compatible, Gain bandwidth 5.5 MHz instead of 3 MHz) Larger power inductor for MC34063.
Parts:
- removed D6: ZD-3V3-SOT23, Diodes_SMD:SOD-123, symbol ZENERsmall-RESCUE-MP-Tracker
- removed R25: 2k2, Resistors_SMD:R_0805, symbol R-RESCUE-MP-Tracker
- added C17, C18: 470n, symbol C-RESCUE-MP-Tracker
- added C19, C23, C24: 470n, ~, symbol C-RESCUE-MP-Tracker
- added D7, D9: 1N4001, Diodes_SMD:SOD-323, symbol DIODE
- added R31, R32: 1K, Resistors_SMD:R_0805, symbol R-RESCUE-MP-Tracker
- added R33, R34: 27k, Resistors_SMD:R_0805, symbol R-RESCUE-MP-Tracker
- added R35, R36: 3k3, Resistors_SMD:R_0805, symbol R-RESCUE-MP-Tracker
- added RV1: 250R, symbol POT
- C10, C16: value 100n -> 470n
- C12, C15, C20, C21, C22: value 10n -> 470n
- C8: value 1n5 -> 68p
- L1: value 22u -> 100u
- R12: value 3k9 -> 3k3
- R17: value 4k7 -> 27k
- R18: value 22k -> 330k
- R19: value 15k -> 10k
- R20: value 47k -> 27k
- R21: value 4k4 -> 2k2
- R22: value 100R -> 69R
- R23: value 10k -> 3k4
- R30: value 1k2 -> 15k
- U2: value TL082 -> MC4558
- gave numbers to parts that had none: 2
Connections:
- wire segments 246 -> 260
Other:
- note added: "Conn \nTempSense"
- note added: "Freifunk-Open-MPP-Solar-Tracker Rev. 2"
- note removed: "Freifunk-Open-MPP-Solar-Tracker"
- note removed: "To Temperature\nSensor"
- moved on the sheet: C10, C12, C15, C16, C20, C21, D3, D4, R10, R11, R12, R13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

Commit message: Update schematic and board design and firmware source.
Parts:
- removed C15, C19, C20, C21, C22, C23, C24: 470n, ~, symbol C-RESCUE-MP-Tracker
- removed D3: ZD-3V3-SOT23, Diodes_SMD:SOD-123, symbol ZENERsmall-RESCUE-MP-Tracker
- removed P1: DIL10, Pin_Headers:Pin_Header_Straight_2x05, symbol DIL10
- removed R17, R33, R34: 27k, Resistors_SMD:R_0805, symbol R-RESCUE-MP-Tracker
- removed R18: 330k, Resistors_SMD:R_0805, symbol R-RESCUE-MP-Tracker
- removed R23: 3k4, Resistors_SMD:R_0805, symbol R-RESCUE-MP-Tracker
- removed R24, R29: 22k, Resistors_SMD:R_0805, symbol R-RESCUE-MP-Tracker
- removed R28: 10k, Resistors_SMD:R_0805, symbol R-RESCUE-MP-Tracker
- removed R30: 15k, Resistors_SMD:R_0805, symbol R-RESCUE-MP-Tracker
- removed R35, R36: 3k3, Resistors_SMD:R_0805, symbol R-RESCUE-MP-Tracker
- removed RV1: 250R, symbol POT
- removed U2: MC4558, Housings_SOIC:SOIC-8-1EP_3.9x4.9mm_Pitch1.27mm, symbol TL082-RESCUE-MP-Tracker
- added P1: CONN_02X05, Pin_Headers:Pin_Header_Straight_2x05, symbol CONN_02X05
- added U2: TL081, Housings_SOIC:SOIC-8_3.9x4.9mm_Pitch1.27mm, symbol TL081
- C1, C10, C17, C18, C2, C3, C4, C5: footprint (none) -> Capacitors_SMD:C_1206_HandSoldering
- C11, C7, C8, C9: footprint (none) -> Capacitors_SMD:C_0805_HandSoldering
- C12, C16: footprint ~ -> Capacitors_SMD:C_1206_HandSoldering
- C13, C14: footprint ~ -> Capacitors_SMD:c_elec_10x10.5
- C6: footprint (none) -> Capacitors_SMD:c_elec_10x10.5
- P2: footprint (none) -> Pin_Headers:Pin_Header_Straight_1x02
- U4: footprint (none) -> Housings_SOIC:SOIC-8-1EP_3.9x4.9mm_Pitch1.27mm
Connections:
- wire segments 260 -> 276
Other:
- note added: "3V3"
- note added: "GND"
- note added: "MISO"
- note added: "MOSI"
- note added: "RESET"
- note added: "RX"
- note added: "SCLK"
- note added: "TX"
- moved on the sheet: C16, R22

Commit message: Updated firmware with temperature sensor support (KTY81-210) Minor fixes in the schematic.
Parts:
- added R17: 1K5, Resistors_SMD:R_0805, symbol R-RESCUE-MP-Tracker
- U2: symbol TL081 -> TL081-RESCUE-MP-Tracker
Connections:
- wire segments 276 -> 282
Other:
- moved on the sheet: C17, R31
